File: hardware/pathA_CM5-DETECT_rev0.3/kicad/CM5-DETECT_rev03_placed.kicad_pcb (KiCad board)
At the start: 4 copper layers, 44 x 134 mm, 192 parts, among them M1 Raspberry Pi CM5 (CM5108032 /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

Commit message: rev0.3: ATECC608B secure element, package builder, RK3576 module model
Co-Authored-By: Claude Opus 5.5 <noreply@anthropic.com>
Claude-Session: https://claude.ai/code/session_01QU2atnSo3eyX8zZazu88cn
Parts:
- added C55: 47uF 16V, C_1210_3225Metric, B.Cu at (35.4, 24.0)
- added U_SEC: ATECC608B secure element (I2C 0x60), SOIC-8_3.9x4.9mm_P1.27mm, B.Cu at (29.8, 26.2)
- C54: value 47uF 16V -> 100nF; footprint C_1210_3225Metric -> C_0402_1005Metric
- moved C54 14.4 mm to (28.1, 11.6)
- moved R26 8.29 mm to (28.4, 14.3), turned to 90 degrees
- moved R27 4.25 mm to (30.4, 6.24), turned to 0 degrees
- moved R33 2.48 mm to (34.6, 7.72)
- moved C7 1.50 mm to (26.2, 11.6)
Connections:
- C54 pad 1: VSERVO -> +3V3_CM5
