File: hardware/pathA_CM5-DETECT_rev0.3/kicad/CM5-DETECT_rev03_placed.kicad_pcb (KiCad board)
At the start: 4 copper layers, 44 x 134 mm, 194 parts, among them M1 Raspberry Pi CM5 (CM5108032 /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

Commit message: rev0.3: board stretched to 44x157 (power section spacing), finisher routers (3-layer A*, GND island vias), DSN helper
Co-Authored-By: Claude Sonnet 5.5 <noreply@anthropic.com>
Claude-Session: https://claude.ai/code/session_01QU2atnSo3eyX8zZazu88cn
Parts:
- moved R1 33.0 mm to (36.6, 153.8), turned to 0 degrees
- moved H1 30.4 mm to (2.00, 112.0)
- moved H2 30.4 mm to (42.0, 112.0)
- moved R24 24.2 mm to (14.1, 78.7)
- moved C39 23.8 mm to (17.5, 85.4)
- moved R19 22.6 mm to (16.3, 72.4), turned to 0 degrees
- moved R12 21.7 mm to (42.6, 95.9), turned to 90 degrees
- moved THERMAL USB 21.5 mm to (3.40, 147.0)
- moved C_BULK 21.0 mm to (24.0, 149.0)
- moved Q_RP 21.0 mm to (36.0, 149.0)
- moved R28 20.9 mm to (35.7, 86.2), turned to 0 degrees
- moved TP_SWIO 20.9 mm to (30.3, 42.9)
- moved R7 20.5 mm to (5.15, 98.0), turned to 0 degrees
- moved XT30 alt 17.9 mm to (11.0, 136.8)
- moved R14 17.6 mm to (42.2, 88.2)
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Other:
- board size 44 x 134 mm -> 44 x 157 mm
